File: 128ch-hdemg-sleeve.kicad_pcb (KiCad board)
At the start: 2 copper layers, 150 parts, among them U130 RHD2164_BGA_BGA, U131 RHD2164_BGA_BGA, U132 74HC4053_TSSOP-16

Commit message: Added Python example and support
Parts:
- added H1: MountingHole_Pad, MountingHole:MountingHole_3.2mm_M3_Pad_TopOnly, F.Cu at (46.0, 81.5)
- added H10: MountingHole_Pad, MountingHole:MountingHole_3.2mm_M3_Pad_TopOnly, F.Cu at (38.0, 81.5)
- added H2: MountingHole_Pad, MountingHole:MountingHole_3.2mm_M3_Pad_TopOnly, F.Cu at (46.0, 89.5)
- added H3: MountingHole_Pad, MountingHole:MountingHole_3.2mm_M3_Pad_TopOnly, F.Cu at (22.1, 73.6)
- added H4: MountingHole_Pad, MountingHole:MountingHole_3.2mm_M3_Pad_TopOnly, F.Cu at (22.1, 81.5)
- added H5: MountingHole_Pad, MountingHole:MountingHole_3.2mm_M3_Pad_TopOnly, F.Cu at (22.1, 89.5)
- added H6: MountingHole_Pad, MountingHole:MountingHole_3.2mm_M3_Pad_TopOnly, F.Cu at (30.1, 73.6)
- added H7: MountingHole_Pad, MountingHole:MountingHole_3.2mm_M3_Pad_TopOnly, F.Cu at (30.1, 81.5)
- added H8: MountingHole_Pad, MountingHole:MountingHole_3.2mm_M3_Pad_TopOnly, F.Cu at (30.1, 89.5)
- added H9: MountingHole_Pad, MountingHole:MountingHole_3.2mm_M3_Pad_TopOnly, F.Cu at (38.0, 73.6)
- added REF.0: TESTPOINT_SMALL, TestPoint:TestPoint_THTPad_1.0x1.0mm_Drill0.5mm, F.Cu at (152.5, 91.0)
- moved U125 78.1 mm to (253.5, 133.0)
- moved U126 77.9 mm to (253.5, 148.0)
- moved U116 58.4 mm to (178.5, 148.0)
- moved U115 58.2 mm to (178.5, 133.0)
- moved U124 51.0 mm to (238.5, 148.0)
- moved U123 50.7 mm to (238.5, 133.0)
- moved U10 41.5 mm to (136.8, 111.2)
- moved U9 40.9 mm to (131.0, 109.6)
- moved U8 40.3 mm to (125.2, 108.1)
- moved U7 39.8 mm to (119.4, 106.5)
- moved U6 39.3 mm to (113.6, 105.0)
- moved U5 38.8 mm to (107.8, 103.4)
- moved U4 38.4 mm to (102.0, 101.9)
- moved U11 38.2 mm to (87.2, 87.5)
- moved U3 38.0 mm to (96.2, 100.3)
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- renumbered H1 to H13, H2 to H14

Commit message: updating remote repo
Parts:
- removed the GND.0 at (173.5, 91.0)
- removed the GND0 at (171.5, 109.5)
- removed H13, H14: MOUNTING_HOLE_60MIL, MountingHole:MountingHole_2.2mm_M2
- removed R0: R_0402, Resistor_SMD:R_0402_1005Metric
- removed R4, R5, R6: R_0201, Resistor_SMD:R_0201_0603Metric
- removed the REF0 at (171.5, 106.0)
- removed U131: RHD2164_BGA_BGA, RHD2000:BGA104_9X7
- removed U132: 74HC4053_TSSOP-16, CustomComponents:TSSOP16
- removed the VDD0 at (171.6, 112.7)
- added GND.0: TESTPOINT_SMALL, TestPoint:TestPoint_THTPad_1.0x1.0mm_Drill0.5mm, F.Cu at (127.4, 90.0)
- added GND.0: TESTPOINT_SMALL, TESTPOINT_SMALL, F.Cu at (171.9, 90.9)
- added GND0: TESTPOINT_SMALL, TestPoint:TestPoint_THTPad_1.0x1.0mm_Drill0.5mm, F.Cu at (127.4, 86.9)
- added GND0: TESTPOINT_SMALL, TESTPOINT_SMALL, F.Cu at (172.1, 118.9)
- added H11: MountingHole_Pad, MountingHole:MountingHole_5.3mm_M5_ISO7380_Pad, F.Cu at (273.0, 124.1)
- added H12: MountingHole_Pad, MountingHole:MountingHole_5.3mm_M5_ISO7380_Pad, F.Cu at (223.1, 91.3)
- added REF0: TESTPOINT_SMALL, TestPoint:TestPoint_THTPad_1.0x1.0mm_Drill0.5mm, F.Cu at (127.4, 93.0)
- added REF0: TESTPOINT_SMALL, TESTPOINT_SMALL, F.Cu at (172.1, 116.3)
- added S1: MOLEX_SLIMSTACK_64, MOLEX_SLIMSTACK_64, F.Cu at (158.8, 97.4)
- added S2: MOLEX_SLIMSTACK_64, MOLEX_SLIMSTACK_64, F.Cu at (167.7, 97.4)
- added SW1: SW_DIP_x01, Button_Switch_SMD:SW_DIP_SPSTx01_Slide_Copal_CVS-01xB_W5.9mm_P1mm, F.Cu at (174.3, 39.9)
- added U129: ~, CustomComponents:1625-5-57-15_D3.18mm_disk, B.Cu at (163.5, 128.0)
- added U138: RHD2164_BGA_BGA, RHD2000:BGA104_9X7, F.Cu at (158.1, 111.0)
- added U139: RHD2164_BGA_BGA, RHD2000:BGA104_9X7, F.Cu at (168.4, 111.0)
- added VDD0: TESTPOINT_SMALL, TESTPOINT_SMALL, F.Cu at (172.1, 122.5)
- added VDD0: TESTPOINT_SMALL, TestPoint:TestPoint_THTPad_1.0x1.0mm_Drill0.5mm, F.Cu at (172.7, 124.7)
- H1, H10, H2, H3, H4, H5, H6, H7, H8, H9: footprint MountingHole:MountingHole_3.2mm_M3_Pad_TopOnly -> MountingHole:MountingHole_5.3mm_M5_ISO7380_Pad
- S4: footprint RHD2000:OMNETICS_PZN-06-AA -> OMNETICS_PZN-06-AA
- U1, U10, U100, U101, U102, U103, U104, U105, U106, U107, U108, U109, U11, U110, U111, U112, U113, U114, U115, U116, U117, U118, U119, U12, U120, U121, U122, U123, U124, U125, U126, U127, U128, U13, U14, U15, U16, U17, U18, U19, U2, U20, U21, U22, U23, U24, U25, U26, U27, U28, U29, U3, U30, U31, U32, U33, U34, U35, U36, U37, U38, U39, U4, U40, U41, U42, U43, U44, U45, U46, U47, U48, U49, U5, U50, U51, U52, U53, U54, U55, U56, U57, U58, U59, U6, U60, U61, U62, U63, U64, U65, U66, U67, U68, U69, U7, U70, U71, U72, U73, U74, U75, U76, U77, U78, U79, U8, U80, U81, U82, U83, U84, U85, U86, U87, U88, U89, U9, U90, U91, U92, U93, U94, U95, U96, U97, U98, U99: moved to B.Cu
- U130: value RHD2164_BGA_BGA -> ~; footprint RHD2000:BGA104_9X7 -> CustomComponents:1625-5-57-15_D3.18mm_disk; moved to B.Cu
- moved H8 197.2 mm to (224.2, 124.1)
- moved U52 180.0 mm to (245.5, 95.0)
- moved U74 177.4 mm to (66.5, 120.0)
- moved U125 177.3 mm to (81.5, 90.0)
- moved U126 176.8 mm to (86.5, 90.0)
- moved U73 176.4 mm to (61.5, 120.0)
- moved U54 175.2 mm to (255.5, 95.0)
- moved U31 173.2 mm to (260.5, 110.0)
- moved U123 172.4 mm to (71.5, 90.0)
- moved U32 172.1 mm to (265.5, 110.0)
- moved U124 172.1 mm to (76.5, 90.0)
- moved U51 171.3 mm to (240.5, 95.0)
- moved U56 170.4 mm to (265.5, 95.0)
- moved U114 169.5 mm to (66.5, 95.0)
- moved U113 168.4 mm to (61.5, 95.0)
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Connections:
- C2 pad 1: Net-(U130-ADC_REF) -> Net-(U139-ADC_REF)
- U14 pad 1: Net-(U130-IN13) -> Net-(U139-IN13)
- U15 pad 1: Net-(U130-IN14) -> Net-(U139-IN14)
- U16 pad 1: Net-(U130-IN15) -> Net-(U139-IN15)
- U17 pad 1: Net-(U130-IN16) -> Net-(U139-IN16)
- U18 pad 1: Net-(U130-IN17) -> Net-(U139-IN17)
- U19 pad 1: Net-(U130-IN18) -> Net-(U139-IN18)
- U2 pad 1: Net-(U130-IN1) -> Net-(U139-IN1)
- U20 pad 1: Net-(U130-IN19) -> Net-(U139-IN19)
- U21 pad 1: Net-(U130-IN20) -> Net-(U139-IN20)
- U22 pad 1: Net-(U130-IN21) -> Net-(U139-IN21)
- U23 pad 1: Net-(U130-IN22) -> Net-(U139-IN22)
- U24 pad 1: Net-(U130-IN23) -> Net-(U139-IN23)
- U25 pad 1: Net-(U130-IN24) -> Net-(U139-IN24)
- U26 pad 1: Net-(U130-IN25) -> Net-(U139-IN25)
- U27 pad 1: Net-(U130-IN26) -> Net-(U139-IN26)
- U28 pad 1: Net-(U130-IN27) -> Net-(U139-IN27)
- U29 pad 1: Net-(U130-IN28) -> Net-(U139-IN28)
- U3 pad 1: Net-(U130-IN2) -> Net-(U139-IN2)
- U30 pad 1: Net-(U130-IN29) -> Net-(U139-IN29)
- U31 pad 1: Net-(U130-IN30) -> Net-(U139-IN30)
- U32 pad 1: Net-(U130-IN31) -> Net-(U139-IN31)
- U33 pad 1: Net-(U130-IN32) -> Net-(U139-IN32)
- U34 pad 1: Net-(U130-IN33) -> Net-(U139-IN33)
- U35 pad 1: Net-(U130-IN34) -> Net-(U139-IN34)
- U36 pad 1: Net-(U130-IN35) -> Net-(U139-IN35)
- U37 pad 1: Net-(U130-IN36) -> Net-(U139-IN36)
- U38 pad 1: Net-(U130-IN37) -> Net-(U139-IN37)
- U39 pad 1: Net-(U130-IN38) -> Net-(U139-IN38)
- U4 pad 1: Net-(U130-IN3) -> Net-(U139-IN3)
- U40 pad 1: Net-(U130-IN39) -> Net-(U139-IN39)
- U41 pad 1: Net-(U130-IN40) -> Net-(U139-IN40)
- U42 pad 1: Net-(U130-IN41) -> Net-(U139-IN41)
- U43 pad 1: Net-(U130-IN42) -> Net-(U139-IN42)
- U44 pad 1: Net-(U130-IN43) -> Net-(U139-IN43)
- U45 pad 1: Net-(U130-IN44) -> Net-(U139-IN44)
- U46 pad 1: Net-(U130-IN45) -> Net-(U139-IN45)
- U47 pad 1: Net-(U130-IN46) -> Net-(U139-IN46)
- U48 pad 1: Net-(U130-IN47) -> Net-(U139-IN47)
- U49 pad 1: Net-(U130-IN48) -> Net-(U139-IN48)
- U5 pad 1: Net-(U130-IN4) -> Net-(U139-IN4)
- U50 pad 1: Net-(U130-IN49) -> Net-(U139-IN49)
- U51 pad 1: Net-(U130-IN50) -> Net-(U139-IN50)
- U52 pad 1: Net-(U130-IN51) -> Net-(U139-IN51)
- U53 pad 1: Net-(U130-IN52) -> Net-(U139-IN52)
- U54 pad 1: Net-(U130-IN53) -> Net-(U139-IN53)
- U55 pad 1: Net-(U130-IN54) -> Net-(U139-IN54)
- U56 pad 1: Net-(U130-IN55) -> Net-(U139-IN55)
- U57 pad 1: Net-(U130-IN56) -> Net-(U139-IN56)
- U58 pad 1: Net-(U130-IN57) -> Net-(U139-IN57)
- U59 pad 1: Net-(U130-IN58) -> Net-(U139-IN58)
- U6 pad 1: Net-(U130-IN5) -> Net-(U139-IN5)
- U60 pad 1: Net-(U130-IN59) -> Net-(U139-IN59)
- U61 pad 1: Net-(U130-IN60) -> Net-(U139-IN60)
- U62 pad 1: Net-(U130-IN61) -> Net-(U139-IN61)
- U63 pad 1: Net-(U130-IN62) -> Net-(U139-IN62)
- U64 pad 1: Net-(U130-IN63) -> Net-(U139-IN63)
- U7 pad 1: Net-(U130-IN6) -> Net-(U139-IN6)
- U8 pad 1: Net-(U130-IN7) -> Net-(U139-IN7)
- U9 pad 1: Net-(U130-IN8) -> Net-(U139-IN8)
Routing:
- net REF: track 0.00 -> 100.2 mm, vias 0 -> 1
- net GND: track 0.00 -> 79.4 mm, vias 0 -> 8
- net N$99: track 0.00 -> 54.5 mm, vias 0 -> 1
- net N$2: track 0.00 -> 49.3 mm, vias 0 -> 1
- net CS-: track 0.00 -> 46.6 mm, vias 0 -> 2
- net N$103: track 0.00 -> 45.1 mm, vias 0 -> 1
- net N$12: track 0.00 -> 44.3 mm, vias 0 -> 1
- net N$8: track 0.00 -> 41.6 mm, vias 0 -> 1
- net VCC: track 0.00 -> 36.2 mm, vias 0 -> 6
- net N$46: track 0.00 -> 35.0 mm, vias 0 -> 1
- net N$48: track 0.00 -> 33.5 mm, vias 0 -> 1
- net N$53: track 0.00 -> 30.6 mm, vias 0 -> 1
- net N$97: track 0.00 -> 29.1 mm, vias 0 -> 1
- net N$101: track 0.00 -> 28.1 mm, vias 0 -> 1
- net N$102: track 0.00 -> 27.8 mm, vias 0 -> 1
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- added copper zone on In2.Cu, net GND
- added copper zone on In1.Cu, net VCC
Other:
- board outline added: 230 x 50 mm
- copper layers 2 -> 4
- board text added: "0"
- board text added: "0-63"
- board text added: "127"
- board text added: "128-channel amplifier board"
- board text added: "31"
- board text added: "32"
- board text added: "63"
- board text added: "64"
- board text added: "64-127"
- board text added: "6mm"
- board text added: "95"
- board text added: "96"
- board text added: "GND"
- board text added: "Intan Technologies"
- board text added: "MOUNT"
- board text added: "REF"
- board text added: "VDD"
- board text added: "www.intantech.com"
